File: NoodleBoard.kicad_sch (KiCad schematic)
At the start: 0 parts

Commit message: feat: setup schematics
Parts:
- added C1, C10, C11, C17, C2, C3, C4, C5, C6, C7, C8: 100n, symbol Device:C
- added C12, C9: 1u, symbol Device:C
- added C13, C14: 10u, symbol Device:C
- added C15, C16: 33p, symbol Device:C
- added J1: USB_C_Receptacle_USB2.0_16P, PCM_marbastlib-various:USB_C_Receptacle_HRO_TYPE-C-31-M-23, symbol Connector:USB_C_Receptacle_USB2.0_16P
- added J2: Left, symbol Connector_Generic:Conn_01x20
- added J3: Right, symbol Connector_Generic:Conn_01x20
- added J4: Middle, symbol Connector_Generic:Conn_01x03
- added J5: Bottom, symbol Connector_Generic:Conn_01x05
- added R1, R2, R5: 5.1k, symbol Device:R
- added R3, R4: 27, symbol Device:R
- added R6: 10k, symbol Device:R
- added R7: 1k, symbol Device:R
- added SW1: SW_Push, symbol Switch:SW_Push_45deg
- added U1: RP2040, Package_DFN_QFN:QFN-56-1EP_7x7mm_P0.4mm_EP3.2x3.2mm, symbol MCU_RaspberryPi:RP2040
- added U2: ME6211C33M5, Package_TO_SOT_SMD:SOT-23-5, symbol Regulator_Linear:ME6211C33M5
- added U3: W25Q128JVS, Package_SO:SOIC-8_5.3x5.3mm_P1.27mm, symbol Memory_Flash:W25Q128JVS
- added Y1: 12MHz, symbol Device:Crystal_GND24
Connections:
- new net: R7.2, SW1.2
- new net: C15.2, R5.1, Y1.3
- new net: J1.A7 (D-), J1.B7 (D-), R3.2
- new net: J1.B5 (CC2), R2.1
- new net: J1.A5 (CC1), R1.1
- new net: J1.A6 (D+), J1.B6 (D+), R4.2
- new net +1V1: C10.1, C11.1, C12.2, U1.23 (DVDD), U1.45 (VREG_VOUT), U1.50 (DVDD)
- new net +3V3: C1.1, C14.2, C17.1, C2.1, C3.1, C4.1, C5.1, C6.1, C7.1, C8.1, C9.2, J3.5 (Pin_5), R6.1, U1.1 (IOVDD), U1.10 (IOVDD), U1.22 (IOVDD), U1.33 (IOVDD), U1.42 (IOVDD), U1.43 (ADC_AVDD), U1.44 (VREG_IN), U1.48 (USB_VDD), U1.49 (IOVDD), U2.5 (V_{OUT}), U3.8 (VCC)
- new net GND: C1.2, C10.2, C11.2, C12.1, C13.1, C14.1, C15.1, C16.1, C17.2, C2.2, C3.2, C4.2, C5.2, C6.2, C7.2, C8.2, C9.1, J1.A1 (GND), J1.A12 (GND), J1.B1 (GND), J1.B12 (GND), J1.S1 (SHIELD), J2.13 (Pin_13), J2.18 (Pin_18), J2.3 (Pin_3), J2.8 (Pin_8), J3.13 (Pin_13), J3.18 (Pin_18), J3.3 (Pin_3), J3.8 (Pin_8), J4.2 (Pin_2), J5.5 (Pin_5), R1.2, R2.2, SW1.1, U1.57 (GND), U2.2 (V_{SS}), U3.4 (GND), Y1.2, Y1.4
- new net GPIO0: J2.1 (Pin_1), U1.2 (GPIO0)
- new net GPIO1: J2.2 (Pin_2), U1.3 (GPIO1)
- new net GPIO10: J2.14 (Pin_14), U1.13 (GPIO10)
- new net GPIO11: J2.15 (Pin_15), U1.14 (GPIO11)
- new net GPIO12: J2.16 (Pin_16), U1.15 (GPIO12)
- new net GPIO13: J2.17 (Pin_17), U1.16 (GPIO13)
- new net GPIO14: J2.19 (Pin_19), U1.17 (GPIO14)
- new net GPIO15: J2.20 (Pin_20), U1.18 (GPIO15)
- new net GPIO16: J3.20 (Pin_20), U1.27 (GPIO16)
- new net GPIO17: J3.19 (Pin_19), U1.28 (GPIO17)
- new net GPIO18: J3.17 (Pin_17), U1.29 (GPIO18)
- new net GPIO19: J3.16 (Pin_16), U1.30 (GPIO19)
- new net GPIO2: J2.4 (Pin_4), U1.4 (GPIO2)
- new net GPIO20: J3.15 (Pin_15), U1.31 (GPIO20)
- new net GPIO21: J3.14 (Pin_14), U1.32 (GPIO21)
- new net GPIO22: J3.12 (Pin_12), U1.34 (GPIO22)
- new net GPIO23: J5.1 (Pin_1), U1.35 (GPIO23)
- new net GPIO24: J5.2 (Pin_2), U1.36 (GPIO24)
- new net GPIO25: J5.3 (Pin_3), U1.37 (GPIO25)
- new net GPIO26_ADC0: J3.10 (Pin_10), U1.38 (GPIO26_ADC0)
- new net GPIO27_ADC1: J3.9 (Pin_9), U1.39 (GPIO27_ADC1)
- new net GPIO28_ADC2: J5.4 (Pin_4), U1.40 (GPIO28_ADC2)
- new net GPIO29_ADC3: J3.7 (Pin_7), U1.41 (GPIO29_ADC3)
- new net GPIO3: J2.5 (Pin_5), U1.5 (GPIO3)
- new net GPIO4: J2.6 (Pin_6), U1.6 (GPIO4)
- new net GPIO5: J2.7 (Pin_7), U1.7 (GPIO5)
- new net GPIO6: J2.9 (Pin_9), U1.8 (GPIO6)
- new net GPIO7: J2.10 (Pin_10), U1.9 (GPIO7)
- new net GPIO8: J2.11 (Pin_11), U1.11 (GPIO8)
- new net GPIO9: J2.12 (Pin_12), U1.12 (GPIO9)
- new net QSPI_SCLK: U1.52 (QSPI_SCLK), U3.6 (CLK)
- new net QSPI_SD0: U1.53 (QSPI_SD0), U3.5 (DI/IO_{0})
- new net QSPI_SD1: U1.55 (QSPI_SD1), U3.2 (DO/IO_{1})
- new net QSPI_SD2: U1.54 (QSPI_SD2), U3.3 (~{WP}/IO_{2})
- new net QSPI_SD3: U1.51 (QSPI_SD3), U3.7 (~{HOLD}/~{RESET}/IO_{3})
- new net QSPI_SS: R6.2, R7.1, U1.56 (QSPI_SS), U3.1 (~{CS})
- new net RUN: J3.11 (Pin_11), U1.26 (RUN)
- new net SWCLK: J4.1 (Pin_1), U1.24 (SWCLK)
- new net SWD: J4.3 (Pin_3), U1.25 (SWD)
- new net TESTEN: U1.19 (TESTEN)
- new net USB_DM: R4.1, U1.46 (USB_DM)
- new net USB_DP: R3.1, U1.47 (USB_DP)
- new net VBUS: C13.2, J1.A4 (VBUS), J1.A9 (VBUS), J1.B4 (VBUS), J1.B9 (VBUS), J3.1 (Pin_1), U2.1 (V_{IN}), U2.3 (CE)
- new net XIN: C16.2, U1.20 (XIN), Y1.1
- new net XOUT: R5.2, U1.21 (XOUT)
- no-connect marks 0 -> 2
Other:
- note added: "1v1 Decoupling"
- note added: "3v3 Decoupling"
- note added: "C12(1u) should be close to the 45th pin !!"
- note added: "C9 (1u) should be close to the 44th pin !!"
- note added: "Connectors"
- note added: "Crystal Oscillator"
- note added: "Flash memory"
- note added: "MCU"
- note added: "R3 and R4 should be close to the RP2040 !!"
- note added: "USB-C"
- note added: "Voltage Regulator"

Commit message: feat: upload v1 pcb and schematics
Parts:
- removed J5: Bottom, symbol Connector_Generic:Conn_01x05
- added J5: Bottom, Connector_PinHeader_2.54mm:PinHeader_1x03_P2.54mm_Vertical, symbol Connector_Generic:Conn_01x03
- added SW2: Reset, Button_Switch_SMD:SW_Push_SPST_NO_Alps_SKRK, symbol Switch:SW_Push_45deg
- C1, C10, C11, C12, C15, C16, C17, C2, C3, C4, C5, C6, C7, C8, C9: footprint (none) -> Capacitor_SMD:C_0402_1005Metric
- C13, C14: footprint (none) -> Capacitor_SMD:C_0603_1608Metric
- J1: footprint PCM_marbastlib-various:USB_C_Receptacle_HRO_TYPE-C-31-M-23 -> PCM_marbastlib-various:USB_C_Receptacle_HRO_TYPE-C-31-M-12
- J2, J3: footprint (none) -> Connector_PinHeader_2.54mm:PinHeader_1x20_P2.54mm_Vertical
- J4: footprint (none) -> Connector_PinHeader_2.54mm:PinHeader_1x03_P2.54mm_Vertical
- R1, R2, R5, R6, R7: footprint (none) -> Resistor_SMD:R_0603_1608Metric
- R3, R4: footprint (none) -> Resistor_SMD:R_0402_1005Metric
- SW1: value SW_Push -> Boot; footprint (none) -> Button_Switch_SMD:SW_Push_SPST_NO_Alps_SKRK
- U3: value W25Q128JVS -> W25Q16JVZPIQ TR; footprint Package_SO:SOIC-8_5.3x5.3mm_P1.27mm -> Package_SON:Winbond_USON-8-1EP_3x2mm_P0.5mm_EP0.2x1.6mm
- Y1: footprint (none) -> Crystal:Crystal_SMD_3225-4Pin_3.2x2.5mm_HandSoldering
Connections:
- net TESTEN is gone; now on net GND: U1.19 (TESTEN)
- net +3V3: now also J5.2 (Pin_2)
- net GND: now also J5.3 (Pin_3), SW2.1
- net GPIO23: now also J3.11 (Pin_11)
- net GPIO24: now also J3.10 (Pin_10)
- net GPIO25: now also J3.9 (Pin_9)
- net GPIO26_ADC0: now also J3.7 (Pin_7); no longer J3.10 (Pin_10)
- net GPIO27_ADC1: now also J3.6 (Pin_6); no longer J3.9 (Pin_9)
- net GPIO28_ADC2: now also J3.4 (Pin_4)
- net GPIO29_ADC3: now also J3.2 (Pin_2); no longer J3.7 (Pin_7)
- net RUN: now also J5.1 (Pin_1), SW2.2; no longer J3.11 (Pin_11)
- net USB_DM renamed USB_D+
- net USB_D+: now also U1.47 (USB_DP); no longer U1.46 (USB_DM)
- net USB_DP renamed USB_D-
- net USB_D-: now also U1.46 (USB_DM); no longer U1.47 (USB_DP)
Other:
- note added: "Switches"
- company: (none) -> sanooj.uk
- title: (none) -> NoodleBoard
- moved on the sheet: C17, J2, J3, J4, R6, R7, SW1, U3

Commit message: feat: add all the files
Parts:
- added D1, D2: LED, LED_SMD:LED_0402_1005Metric, symbol Device:LED
- added R8, R9: 1k, Resistor_SMD:R_0402_1005Metric, symbol Device:R
- R5: value 5.1k -> 1k; footprint Resistor_SMD:R_0603_1608Metric -> Resistor_SMD:R_0402_1005Metric
- R7: footprint Resistor_SMD:R_0603_1608Metric -> Resistor_SMD:R_0402_1005Metric
Connections:
- net +3V3: now also R9.2
- net GND: now also D1.1 (K), D2.1 (K)
- net VBUS: now also R8.2
- new net: D1.2 (A), R8.1
- new net: D2.2 (A), R9.1
Other:
- note added: "Power LEDs"
- moved on the sheet: R7, SW1, SW2
